File: Current Iteration/Schematic Layout & PCB/NixieControllerFinal-PHILO.kicad_sch (KiCad schematic)
At the start: 86 parts, among them J1 Conn_01x10_Pin, J2 USB_C_Receptacle_2.0, J3 Conn_01x10_Pin, J4 Conn_01x10_Pin, J5 Conn_01x10_Pin, J6 Conn_01x02, J7 Micro_SD_Card_Det1, J8 Conn_ARM_JTAG_SWD_10, J9 NixieIN, SW1 PEC11J-9215F-S0015, SW5 PEC16-2015F-N0024, SW6 PEC16-2015F-N0024, U1 HV5622PG, U10 NID1100, U11 TPS61040DBV, U13 STM32G0B1KEU6, U14 CM1224-04MR, U2 HV5622PG, U3 4504, U4 CM1224-04MR, U5 NCH6100HV, U6 CAP1206-x-SL, U7 NID1100, U8 MCP1700x-330xxTT, U9 MAX98357A

Commit message: Organization and CAD files
Parts:
- added J10: Conn_01x07_Socket, symbol Connector:Conn_01x07_Socket
- added J11: Conn_01x03_Socket, symbol Connector:Conn_01x03_Socket
- added J12, J13, J14: Conn_01x02_Socket, symbol Connector:Conn_01x02_Socket
- SW1: value PEC11J-9215F-S0015 -> ~; footprint footprints:PEC09-2xxxF-Sxxxx -> Rotary_Encoder:RotaryEncoder_Bourns_Vertical_PEC12R-3x17F-Sxxxx
- SW5, SW6: value PEC16-2015F-N0024 -> ~; footprint footprints:PEC09-2xxxF-Sxxxx -> Rotary_Encoder:RotaryEncoder_Bourns_Vertical_PEC12R-3x17F-Sxxxx
Connections:
- net +5V: no longer D3.1 (K), J2.A4 (VBUS), J2.A9 (VBUS), J2.B4 (VBUS), J2.B9 (VBUS)
- net GND: now also D3.1 (K), J2.A4 (VBUS), J2.A9 (VBUS), J2.B4 (VBUS), J2.B9 (VBUS), J14.1 (Pin_1), J14.2 (Pin_2)
- net ROT1A: now also J10.7 (Pin_7); no longer C16.1, R29.2
- net ROT1B: now also J10.6 (Pin_6); no longer C15.1, R18.1
- net ROT2A: now also J10.5 (Pin_5); no longer C11.1, R21.2
- net ROT2B: now also J10.4 (Pin_4); no longer C12.1, R22.1
- net ROT3A: now also J10.3 (Pin_3); no longer C14.1, R26.2
- net ROT3B: now also J10.2 (Pin_2); no longer C13.1, R23.1
- net SELECT_RET: now also J10.1 (Pin_1), J11.1 (Pin_1)
- new net: C11.1, J12.2 (Pin_2), R21.2
- new net: C15.1, J11.2 (Pin_2), R18.1
- new net: C12.1, J12.1 (Pin_1), R22.1
- new net: C13.1, J13.1 (Pin_1), R23.1
- new net: C16.1, J11.3 (Pin_3), R29.2
- new net: C14.1, J13.2 (Pin_2), R26.2
Other:
- company: (none) -> Author: Fern Potter
- title: (none) -> HV Display Tube Alarm Clock
- moved on the sheet: BT1, C1, C11, C12, C13, C14, C15, C16, C17, C19, C21, C27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

Commit message: repo refresh
Parts:
- removed J10: Conn_01x07_Socket, symbol Connector:Conn_01x07_Socket
- removed J11: Conn_01x03_Socket, symbol Connector:Conn_01x03_Socket
- removed J12, J13, J14: Conn_01x02_Socket, symbol Connector:Conn_01x02_Socket
- removed J2: USB_C_Receptacle_2.0, footprints:12402012E212A_AMP, symbol Connector:USB_C_Receptacle_USB2.0_14P
- added C31: 1uF, Capacitor_SMD:C_0805_2012Metric_Pad1.18x1.45mm_HandSolder, symbol Device:C
- added J10: 2480803-1, Connector_USB:24808031, symbol 24808:2480803-1
- added J11: Conn_01x04_Socket, Connector_JST:JST_SH_BM04B-SRSS-TB_1x04-1MP_P1.00mm_Vertical, symbol Connector:Conn_01x04_Socket
- added J12, J13: Conn_01x03_Socket, Connector_JST:JST_SH_BM03B-SRSS-TB_1x03-1MP_P1.00mm_Vertical, symbol Connector:Conn_01x03_Socket
- added J15: Conn_01x02_Socket, Connector_JST:JST_EH_B2B-EH-A_1x02_P2.50mm_Vertical, symbol Connector:Conn_01x02_Socket
- added J16: Conn_01x08_Socket, Connector_JST:JST_SH_BM08B-SRSS-TB_1x08-1MP_P1.00mm_Vertical, symbol Connector:Conn_01x08_Socket
- added J2: Conn_01x02, symbol Connector_Generic:Conn_01x02
- BT1: footprint (none) -> Connector_JST:JST_EH_B2B-EH-A_1x02_P2.50mm_Vertical
Connections:
- net +3.3V: no longer C19.1, R13.1, R14.1, R6.1, U6.7 (VDD)
- net +5V: now also J15.1 (Pin_1); no longer U14.3 (VP)
- net +V_CRIT: now also C19.1, R13.1, R14.1, R6.1, U6.7 (VDD), U9.2 (GAIN_SLOT), C31.1
- net CC1: now also J10.A5
- net CC2: now also J10.B5
- net GND: now also C31.2, J10.A12, J10.B12, J10.MH1, J10.MH2, J15.2 (Pin_2), J16.8 (Pin_8); no longer C11.2, C12.2, C13.2, C14.2, C15.2, C16.2, D3.1 (K), D3.2 (A), R3.2, R4.2, SW1.C, SW1.S1, SW5.C, SW6.C, U14.8 (VN)
- net ROT1A: now also J16.7 (Pin_7)
- net ROT1B: now also J16.6 (Pin_6)
- net ROT2A: now also J16.5 (Pin_5)
- net ROT2B: now also U13.11 (PA4), J16.4 (Pin_4)
- net ROT3A: now also J16.3 (Pin_3)
- net ROT3B: now also J16.2 (Pin_2)
- net SELECT_RET: now also J16.1 (Pin_1); no longer SW1.S2
- net at C11.1, R21.2: now also J13.2 (Pin_2)
- net HV_Vin2: now reaches J9.3 (Pin_3), R25.2
- net HV_Vin3: now reaches J9.2 (Pin_2), R24.2
- net HV_Vin4: now reaches J9.1 (Pin_1), R20.2
- net at C15.1, R18.1: now also J11.2 (Pin_2)
- net at C12.1, R22.1: now also J13.1 (Pin_1)
- net at C13.1, R23.1: now also J12.1 (Pin_1)
- net at C16.1, R29.2: now also J11.3 (Pin_3)
- net at C14.1, R26.2: now also J12.2 (Pin_2)
- net CS_IN2: now reaches J6.1 (Pin_1), U6.13 (CS2)
- net CS_IN1: now reaches J6.2 (Pin_2), U6.2 (CS1)
- net HV_Vin1: now reaches J9.4 (Pin_4), R27.2
- net SWO: no longer names the net of J8.6 (SWO/TDO)
- new net: C11.2, C12.2, J13.3 (Pin_3), SW5.C
- new net: C15.2, C16.2, J11.4 (Pin_4), SW1.C, SW1.S1
- new net: J11.1 (Pin_1), SW1.S2
- new net: C13.2, C14.2, J12.3 (Pin_3), SW6.C
- new net 5V_IN: D3.1 (K), J10.A9, J10.B9, J2.1 (Pin_1), U14.3 (VP)
- new net GND1: D3.2 (A), J2.2 (Pin_2), R3.2, R4.2, U14.8 (VN)
- no-connect marks 45 -> 41
Other:
- note removed: "r1/r2=9.056 Vout=12.4"
- moved on the sheet: J6, J9

Commit message: Latest PCB revision
Parts:
- added C32: 10uF, Capacitor_SMD:C_1206_3216Metric_Pad1.33x1.80mm_HandSolder, symbol Device:C
- added C33: 0.01uF, Capacitor_SMD:C_0805_2012Metric_Pad1.18x1.45mm_HandSolder, symbol Device:C
- added R1: 10k, Resistor_SMD:R_0805_2012Metric_Pad1.20x1.40mm_HandSolder, symbol Device:R
- added R2: 35K, Resistor_SMD:R_0805_2012Metric_Pad1.20x1.40mm_HandSolder, symbol Device:R
- C27, C28: value 0.1u -> 1uF
- C29, C30: value 0.33u -> 10uF
- C5: value 22uF -> 220uF
Connections:
- net +3.3V: now also R2.1
- net +V_CRIT: now also C32.1
- net GND: now also C32.2
- net at C15.2, C16.2, J11.4 (Pin_4)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: now also R1.2; no longer SW1.S1
- net at J11.1 (Pin_1), SW1.S2: now also C33.1
- net at U10.4 (ST): now also U13.22 (PA11[PA9]), R2.2
- net ~{RESET} renamed ~{JTAG_RST}
- new net: C33.2, R1.1, SW1.S1
- no-connect marks 41 -> 40
Other:
- note added: "--------NC --NC --NC -----VDD -----GND --JTAG_RST -------EXTI0 -------GPIO ----SPI1_MOSI -------EXTI3 -------EXTI4 -----SPI1_SCK -----I2C2_SDA -----I2C2_SCL -----SPI1_NSS -------EXTI1"
- note added: "COULD BE HIGHER TO 80K"
- note added: "I2S2_CK----- I2S2_SD----- GPIO------- EXTI5------- SPI1_MISO---- GPIO------- GPIO------ JTAG_CLK JTAG_IO----- GPIO--- GPIO---- EXTI10----- EXTI6------ EXTI9------ I2S2_WS----- I2S2_MCK----"
- note removed: "SPI1_MISO, I2C2_SCL, I2S1_MCK"
- note removed: "SPI1_MISO, I2C2_SDA, I2C3_SDA,I2S1_MCK"
- note removed: "SPI1_MISO, I2C3_SDA, I2C2_SDA, SPI3_MISO, I2S1_MCK"
- note removed: "SPI1_MOSI, I2C1_SMBA, SPI3_MOSI, I2S1_SD"
- note removed: "SPI1_MOSI, I2C2_SCL, I2C3_SCL,I2S1_SD"
- note removed: "SPI1_MOSI, I2C2_SDA, I2S1_SD, I2S_CKIN"
- note removed: "SPI1_MOSI,I2S1_SD"
- note removed: "SPI1_NSS, I2C2_SMBA, SPI3_NSS, I2S1_WS"
- note removed: "SPI1_NSS,I2S1_WS"
- note removed: "SPI1_NSS,SPI2_MOSI,SPI3_NSS,I2S1_WS,I2S2_SD"
- note removed: "SPI1_SCK, I2C3_SCL, I2C2_SCL, SPI3_SCK, I2S1_CK"
- note removed: "SPI1_SCK, I2S1_CK"
- note removed: "SPI1_SCK,I2S1_CK"
- note removed: "SPI2_MISO, I2C1_SCL, I2C2_SCL, I2S2_MCK"
- note removed: "SPI2_MISO, I2C1_SCL, I2S2_MCK"
- note removed: "SPI2_MISO,I2S2_MCK"
- note removed: "SPI2_MOSI, I2C1_SDA, I2C2_SDA, I2S2_SD"
- note removed: "SPI2_MOSI, I2C1_SDA, I2S2_SD"
- note removed: "SPI2_NSS, I2C1_SDA, I2S2_WS"
- note removed: "SPI2_NSS, I2S2_WS"
- note removed: "SPI2_SCK, I2C1_SCL, I2S2_CK"
- note removed: "SPI2_SCK,I2S2_CK"
- moved on the sheet: C5, LS1, R12, R19, R20, R24, R25, R27
