File: Current Iteration/Schematic Layout & PCB/NixieControllerFinal-PHILO.kicad_sch (KiCad schematic)
At the start: 96 parts, among them J1 Conn_01x10_Pin, J11 Conn_01x04_Socket, J12 Conn_01x03_Socket, J13 Conn_01x03_Socket, J16 Conn_01x08_Socket, J2 JST_EH_B4B, J3 Conn_01x10_Pin, J4 Conn_01x10_Pin, J5 Conn_01x10_Pin, J6 Conn_01x02, J7 Micro_SD_Card_Det1, J8 Conn_ARM_JTAG_SWD_10, J9 NixieIN, U1 HV5622PG, U10 NID1100, U11 TPS61040DBV, U13 STM32G0B1KEU6, U14 CM1224-04MR, U2 HV5622PG, U3 4504, U4 CM1224-04MR, U5 NCH6100HV, U6 CAP1206-x-SL, U7 NID1100, U8 MCP1700x-330xxTT, U9 MAX98357A

Commit message: Updated Readme with improved  firmware documentation/updated src code
Parts:
- removed C5: 220uF, Capacitor_SMD:C_1206_3216Metric_Pad1.33x1.80mm_HandSolder, symbol Device:C
- removed J8: Conn_ARM_JTAG_SWD_10, Connector_JST:JST_SH_BM05B-SRSS-TB_1x05-1MP_P1.00mm_Vertical, symbol Connector:Conn_ARM_JTAG_SWD_10
- removed R2: 35K, Resistor_SMD:R_0805_2012Metric_Pad1.20x1.40mm_HandSolder, symbol Device:R
- removed U7: NID1100, Package_TO_SOT_SMD:SC-74A-5_1.55x2.9mm_P0.95mm, symbol Analog_Switch:MAX40200AUK
- added C32, C35, C36: 0.1uF, Capacitor_SMD:C_0603_1608Metric_Pad1.08x0.95mm_HandSolder, symbol Device:C
- added C37: 220uF Electrolytic, Capacitor_THT:CP_Radial_D5.0mm_P2.00mm, symbol Device:C
- added J10: Conn_ARM_SWD_TagConnect_TC2030, Connector_PinHeader_2.54mm:PinHeader_1x05_P2.54mm_Vertical, symbol Connector:Conn_ARM_SWD_TagConnect_TC2030
- added U12: NID5100, Package_TO_SOT_SMD:SC-74-6_1.55x2.9mm_P0.95mm, symbol Analog_Switch:MAX40200AUK
- C17, C18, C2, C21, C25, C7, C8: footprint Capacitor_SMD:C_0805_2012Metric_Pad1.18x1.45mm_HandSolder -> Capacitor_SMD:C_0603_1608Metric_Pad1.08x0.95mm_HandSolder
- C20, C23: footprint Capacitor_SMD:C_1808_4520Metric_Pad1.72x2.30mm_HandSolder -> Capacitor_SMD:C_0603_1608Metric_Pad1.08x0.95mm_HandSolder
- C24, C6: footprint Capacitor_SMD:C_1206_3216Metric_Pad1.33x1.80mm_HandSolder -> Capacitor_SMD:C_0805_2012Metric_Pad1.18x1.45mm_HandSolder
- C29: footprint Capacitor_SMD:C_0805_2012Metric_Pad1.18x1.45mm_HandSolder -> Capacitor_SMD:C_1206_3216Metric_Pad1.33x1.80mm_HandSolder
- C30: value 10uF -> 10uF 10V; footprint Capacitor_SMD:C_0805_2012Metric_Pad1.18x1.45mm_HandSolder -> Capacitor_SMD:C_0603_1608Metric_Pad1.08x0.95mm_HandSolder
- D1: value 3.3V+ -> 150060AS75000
- D4: value 12V+ -> 150060AS75000
- D5: value 170V+ -> 150060AS75000
- J6: footprint Connector_JST:JST_ZH_B2B-ZR_1x02_P1.50mm_Vertical -> Connector_JST:JST_PH_B2B-PH-K_1x02_P2.00mm_Vertical
- J7: footprint footprints:MEM2061-01-188-00-A_GCT -> Connector_Card:microSD_HC_Molex_104031-0811
- R15: value 670 20% -> 2400 20%
- R16, R17: footprint Resistor_SMD:R_0805_2012Metric_Pad1.20x1.40mm_HandSolder -> Resistor_SMD:R_0603_1608Metric_Pad0.98x0.95mm_HandSolder
- R19: value 11200 20% -> 34k 10%; footprint Resistor_SMD:R_0805_2012Metric_Pad1.20x1.40mm_HandSolder -> Resistor_SMD:R_1206_3216Metric_Pad1.30x1.75mm_HandSolder
- R5: value 86 20% -> 660 20%
- SI1: footprint (none) -> Package_TO_SOT_SMD:SOT-23-5_HandSoldering
- U10: value NID1100 -> NID5100; footprint Package_TO_SOT_SMD:SC-74A-5_1.55x2.9mm_P0.95mm -> Package_TO_SOT_SMD:SC-74-6_1.55x2.9mm_P0.95mm
- U14, U4: footprint Package_SO:MSOP-10_3x3mm_P0.5mm -> Package_SO:TSSOP-10_3x3mm_P0.5mm
Connections:
- net +12V: no longer C25.2
- net +3.3V: now also C25.1; no longer C22.1, U10.3 (EN)
- net +V_CRIT: now also C22.1, U10.6 (OUT), C35.1, C36.1, C37.1, J10.1 (VCC), U12.6 (OUT); no longer U10.5 (OUT)
- net GND: now also C25.2, U10.3 (_EN), C32.2, C35.2, C36.2, C37.2, J10.5 (GND), U12.2 (GND), U12.3 (_EN); no longer C25.1
- net SWCLK: now also J10.4 (SWCLK)
- net SWDIO: now also J10.2 (SWDIO)
- net ~{JTAG_RST}: now also J10.3 (~{RESET})
- net PB: now reaches C33.1, J11.1 (Pin_1), SW1.S2
- net ROT_3A: now reaches C11.1, J13.2 (Pin_2), R21.2
- net GNDC: now reaches C11.2, C12.2, J13.3 (Pin_3), SW5.C
- net at U10.4 (NC): no longer U13.22 (PA11[PA9])
- net GNDA: now reaches C15.2, C16.2, J11.4 (Pin_4), R1.2, SW1.C
- net ROT_2B: now reaches C15.1, J11.2 (Pin_2), R18.1
- net at BT1.1 (+), C27.1: now also C32.1, U12.1 (VDD)
- net ROT_3B: now reaches C12.1, J13.1 (Pin_1), R22.1
- net ROT_1B: now reaches C13.1, J12.1 (Pin_1), R23.1
- net GNDB: now reaches C13.2, C14.2, J12.3 (Pin_3), SW6.C
- net ROT_1A: now reaches C14.1, J12.2 (Pin_2), R26.2
- net ROT_2A: now reaches C16.1, J11.3 (Pin_3), R29.2
- new net: U10.5 (ST), U13.22 (PA11[PA9])
- no-connect marks 39 -> 40
Other:
- note removed: "COULD BE HIGHER TO 80K"
- moved on the sheet: BT1, C22, C29
